File: Project_sapr.kicad_sch (KiCad schematic)
At the start: 0 parts

Commit message: Новая версия библиотеки
Parts:
- added C1, C10, C11, C12, C13, C14, C15, C16, C17, C18, C19, C2, C20, C21, C22, C23, C24, C25, C26, C27, C28, C29, C3, C30, C31, C32, C33, C34, C4, C5, C6, C7, C8, C9: (no value), symbol UGO:C_gost
- added DA1: (no value), symbol UGO:MDS01L-05N
- added DA2: (no value), symbol UGO:ISOUSB
- added DA3: ADP5071AREZ, symbol UGO:ADP5071
- added DA4: (no value), symbol UGO:LM3671M-ADJ
- added DA5: (no value), symbol UGO:ADP2301AUJZ-R7
- added DA6: (no value), symbol UGO:TPS7A4901DGNR
- added DA7: (no value), symbol UGO:TPS7A3001DGNR
- added R1, R10, R11, R12, R13, R14, R15, R16, R17, R18, R19, R2, R3, R4, R5, R6, R7, R8, R9: (no value), symbol UGO:R_gost

Commit message: Обновлена версия библиотеки в проекте
Parts:
- C2: value (none) -> 47000
- C3: value (none) -> 68000
- C4: value (none) -> 1мк
- R2: value (none) -> 12к
- R3: value (none) -> 15к
Connections:
- net at C2.2: now also R2.1
- net at DA3.10 (SS): now also DA3.4 (SYNC/FREQ), DA3.6 (SLEW)
- net at DA3.12 (COMP2): now also R3.2
- net at DA3.16 (VREG): now also C4.2
- net at DA3.17 (PVIN1): now also C5.2, DA3.18 (PVINSYS), DA3.19 (PVIN2)
- net at DA3.8 (COMP1): now also R2.2
- net at C3.2: now also R3.1
- no-connect marks 0 -> 1
Other:
- moved on the sheet: C2, C3, C4, C5, DA3, R2, R3, R5

Commit message: Обновлена версия библиотеки в проекте
Parts:
- added L1: 47мкГн, symbol UGO:L_throttle
- added L2, L5: 6,8мк, symbol UGO:L_gost
- added L3: 15мк, symbol UGO:L_gost
- added L4: 2,2мк, symbol UGO:L_gost
- added VD1: SS24FL, symbol UGO:VD_gost
- added VD2, VD3: DFLS240-7, symbol UGO:VD_gost
- added VD4: B230A-13-F, symbol UGO:VD_gost
- added XT1: (no value), symbol UGO:47346-0001
- added XT2, XT3: (no value), symbol UGO:DS-1021-1x6
- C1, C20: value (none) -> 4,7мк
- C12, C16, C17, C21, C22, C23, C26, C27, C31, C32, C33, C34, C5, C8: value (none) -> 10мк
- C24, C25: value (none) -> 1000
- C28: value (none) -> 0,1мк
- C29: value (none) -> 6,8
- C30: value (none) -> 33
- C6: value (none) -> 22мк
- C7, C9: value (none) -> 1мк
- R1: value (none) -> 5,1
- R10: value (none) -> 56к
- R11: value (none) -> 4,7к
- R12, R14: value (none) -> 12к
- R13, R15: value (none) -> 1к
- R16: value (none) -> 562к
- R17: value (none) -> 100к
- R18: value (none) -> 52,3к
- R19: value (none) -> 10к
- R4: value (none) -> 1Г
- R5: value (none) -> 0
- R6: value (none) -> 110мк
- R7: value (none) -> 2,32М
- R8: value (none) -> 2,43М
- R9: value (none) -> 127к
Connections:
- net at R6.1: now also DA3.13 (FB2), R7.1
- net at R6.2: now also C9.1, DA3.14 (VREF)
- net at C28.1: now also DA5.1 (BST)
- net at C28.2: now also DA5.6 (SW), L5.1, VD4.
- net -16B: now reaches R7.2
- net -16B: now also C17.2, C23.1, DA7.5 (EN), DA7.8 (VIN), VD3.
- net at R1.1: now also C1.1, DA2.1 (VBUS1)
- net GND 2: now reaches R5.1
- net GND 2: now also C12.2, C16.2, C17.1, C21.2, C33.2, C34.2, C5.1, C8.2, DA1.5 (-Vout), DA5.2 (GND), R11.2, R19.2, R4.2, L3.2, VD4., XT2.6, XT3.5, XT3.6
- net GND 3: now reaches R5.2
- net GND 3: now also C2.1, C22.2, C23.2, C24.2, C25.2, C3.1, C31.2, C32.2, C4.1, C9.2, DA3.1 (PGND), DA3.10 (SS), DA3.15 (AGND), DA3.21 (EP(AGND)), DA3.4 (SYNC/FREQ), DA3.6 (SLEW), DA6.4 (GND), DA7.4 (GND), R15.2
- net +15B: now reaches R14.1
- net +15B: now also C21.1, C26.1, C27.1, C31.1, C32.1, DA5.5 (VIN), DA6.1 (VOUT), DA7.1 (VOUT), R10.1, R12.1, XT3.2
- net at R14.2: now also C27.2, DA7.2 (FB), R15.1
- net at DA7.6 (NR/SS): now also C25.1
- net at R10.2: now also DA5.4 (EN), R11.1
- net at C7.1: now also DA2.5 (VCC1)
- net GND 1: now reaches C7.2
- net GND 1: now also C1.2, C6.2, DA1.2 (-Vin), DA2.12 (GND1), DA2.3 (GND1), DA2.9 (EQ10), R4.1, XT1.5
- net +3,3B: now reaches R16.1
- net +3,3B: now also C29.1, C33.1, DA2.16 (CDPENZ2), DA2.20 (EQ20), DA2.27 (V3P3V2), DA2.28 (VBUS2), L4.2, XT3.4
- net at R16.2: now also C29.2, C30.1, DA4.4 (FB), R17.1
- net at R12.2: now also C26.2, DA6.2 (FB), R13.1
- net +5B: now reaches C5.2, DA3.17 (PVIN1), DA3.18 (PVINSYS), DA3.19 (PVIN2)
- net +5B: now also C12.1, C20.1, C34.1, DA4.1 (VIN), DA4.3 (EN), R18.1, L1.2, L5.2, VD1., XT2.1, XT3.1
- net at DA3.2 (SW1): now also L2.2, VD2.
- net at DA3.20 (SW2): now also L3.1, VD3.
- net at DA3.3 (INBK): now also L2.1
- net at DA3.7 (FB1): now also R8.2, R9.1
- net at C20.2: now also DA4.2 (GND)
- net at C24.1: now also DA6.6 (NR/SS)
- net at C30.2: now also R17.2
- net at R18.2: now also DA5.3 (FB), R19.1
- net at DA4.5 (SW): now also L4.1
- net at DA1.1 (+Vin): now also C6.1, VD1.
- net at DA1.7 (+Vout): now also C8.1, L1.1
- net +16B: now reaches C16.1
- net +16B: now also C22.1, DA6.5 (EN), DA6.8 (VIN), R8.1, VD2.
- net at DA2.19 (EQ21): now also DA2.26 (GND2)
- net OTG_FS_DP: now reaches DA2.21 (DD+)
- net OTG_FS_DP: now also XT2.3
- net OTG_FS_DM: now reaches DA2.22 (DD-)
- net OTG_FS_DM: now also XT2.2
- net at DA2.24 (VCC2): now also DA2.25 (V1P8V2)
- new net -15B: XT3.3
- new net SUP_NEG_EN: XT2.5
- new net SUP_POS_EN: XT2.4
- new net UD_N: XT1.2
- new net UN_P: XT1.3
- no-connect marks 1 -> 9
Other:
- company: (none) -> МГТУ им. Баумана
- title: (none) -> Блок питания
- moved on the sheet: C1, C10, C11, C12, C13, C14, C15, C16, C17, C18, C19, C2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

Commit message: Финальная сборка
Parts:
- removed XT2, XT3: (no value), symbol UGO:DS-1021-1x6
- added XT2: (no value), symbol UGO:DS-1021-1x6_1
- added XT3: (no value), symbol UGO:DS-1021-1x6_2
- C1, C20: footprint (none) -> SAPR:C_0201_0603Metric; Manufacturer_Part_Number (none) -> GRM188Z71C475KE21D
- C10: value (none) -> 4,7мк; footprint (none) -> SAPR:C_0201_0603Metric; Manufacturer_Part_Number (none) -> GRM188Z71C475KE21D
- C11, C13: value (none) -> 0,01мк; footprint (none) -> SAPR:C_0201_0603Metric; Manufacturer_Part_Number (none) -> GRM033R71E103KE14D
- C12: footprint (none) -> SAPR:R_0402_1005Metric; Manufacturer_Part_Number (none) -> CC0402MRX5R6BB106
- C14, C15: value (none) -> 0,1мк; footprint (none) -> SAPR:C_0201_0603Metric; Manufacturer_Part_Number (none) -> GRM033Z71C104KE14D
- C16, C17: footprint (none) -> SAPR:C_1210_3225Metric; Manufacturer_Part_Number (none) -> GRM32ER71H106KA12L
- C18, C19: value (none) -> 2,2мк; footprint (none) -> SAPR:C_0201_0603Metric; Manufacturer_Part_Number (none) -> GRM188R71A225KE15D
- C2: footprint (none) -> SAPR:C_0201_0603Metric; Manufacturer_Part_Number (none) -> GCJ188R71E473KA01D
- C21, C26, C27, C34, C5, C8: footprint (none) -> SAPR:C_0402_1005Metric; Manufacturer_Part_Number (none) -> CC0402MRX5R6BB106
- C22, C23, C31, C32: footprint (none) -> SAPR:C_1206_3216Metric; Manufacturer_Part_Number (none) -> GRM31CR61H106KA12L
- C24, C25: footprint (none) -> SAPR:C_0402_1005Metric; Manufacturer_Part_Number (none) -> GCM155R71H102KA37J
- C28: footprint (none) -> SAPR:C_0201_0603Metric; Manufacturer_Part_Number (none) -> GRM033Z71C104KE14D
- C29: footprint (none) -> SAPR:C_0402_1005Metric; Manufacturer_Part_Number (none) -> CC0402CRNPO9BN6R8
- C3: footprint (none) -> SAPR:C_0201_0603Metric; Manufacturer_Part_Number (none) -> GRM188R71H683KA93D
- C30: footprint (none) -> SAPR:C_0402_1005Metric; Manufacturer_Part_Number (none) -> GRM1555C1H330J
- C33: footprint (none) -> SAPR:C_0805_2012Metric; Manufacturer_Part_Number (none) -> GRM21BR60J106K
- C4, C7, C9: footprint (none) -> SAPR:C_0201_0603Metric; Manufacturer_Part_Number (none) -> GRM033R60J105MEA2D
- C6: footprint (none) -> SAPR:C_0402_1005Metric; Manufacturer_Part_Number (none) -> GRM155R60J226ME11D
- DA1: value (none) -> MDS01L-N; footprint (none) -> SAPR:MDS01L-N; Manufacturer_Part_Number (none) -> MDS01L-05N
- DA2: value (none) -> ISOUSB211; footprint (none) -> SAPR:SSOP-28-ISOUSB211; Manufacturer_Part_Number (none) -> ISOUSB211DPR
- DA3: footprint (none) -> SAPR:TSSOP-20_4.4x6.5mm_P0.65mm; Manufacturer_Part_Number (none) -> ADP5071AREZ
- DA4: value (none) -> LM3671MF-ADJ; footprint (none) -> SAPR:SOT-23-5; Manufacturer_Part_Number (none) -> LM3671MF-ADJ
- DA5: value (none) -> ADP2301AUJZ-R7; footprint (none) -> SAPR:TSOT-23-6
- DA6: value (none) -> TPS7A4901DGNR; footprint (none) -> SAPR:MSOP-8-1EP_3x3mm_P0.65mm_EP1.95x2.15mm; Manufacturer_Part_Number (none) -> TPS7A4901DGNR
- DA7: value (none) -> TPS7A3001DGNR; footprint (none) -> SAPR:MSOP-8-1EP_3x3mm_P0.65mm_EP1.95x2.15mm; Manufacturer_Part_Number (none) -> TPS7A3001DGNR
- L1: footprint (none) -> SAPR:L_TDK_NLV32_3.2x2.5mm; Manufacturer_Part_Number (none) -> NLCV32T-470K-EF
- L2, L5: footprint (none) -> SAPR:L_0201_0603Metric; Manufacturer_Part_Number (none) -> MLF1608E6R8KTD25
- L3: footprint (none) -> SAPR:L_0201_0603Metric; Manufacturer_Part_Number (none) -> MLF1608C150KTA00
- L4: footprint (none) -> SAPR:L_0201_0603Metric; Manufacturer_Part_Number (none) -> ILSB0603ER2R2K
- R1: footprint (none) -> SAPR:R_0402_1005Metric; Manufacturer_Part_Number (none) -> RC0402FR-075R1L
- R10: footprint (none) -> SAPR:R_0402_1005Metric; Manufacturer_Part_Number (none) -> RC0402FR-0756KL
- R11: footprint (none) -> SAPR:R_0402_1005Metric; Manufacturer_Part_Number (none) -> RC0402FR-074K7L
- R12, R14, R2: footprint (none) -> SAPR:R_0402_1005Metric; Manufacturer_Part_Number (none) -> RC0402FR-0712KL
- R13, R15: footprint (none) -> SAPR:R_0402_1005Metric; Manufacturer_Part_Number (none) -> RC0402FR-071KL
- R16: footprint (none) -> SAPR:R_0402_1005Metric; Manufacturer_Part_Number (none) -> RC0402FR-07562K
- R17: footprint (none) -> SAPR:R_0402_1005Metric; Manufacturer_Part_Number (none) -> RC0402FR-07100KL
- R18: footprint (none) -> SAPR:R_0402_1005Metric; Manufacturer_Part_Number (none) -> RC0402FR-0752K3L
- R19: footprint (none) -> SAPR:R_0402_1005Metric; Manufacturer_Part_Number (none) -> RC0402FR-0710KL
- R3: footprint (none) -> SAPR:R_0402_1005Metric; Manufacturer_Part_Number (none) -> RC0402FR-0715RL
- R4: footprint (none) -> SAPR:R_1206_3216Metric; Manufacturer_Part_Number (none) -> CRHV1206AF1G00FKET
- R5: footprint (none) -> SAPR:R_0201_0603Metric; Manufacturer_Part_Number (none) -> RC0201FR-070RL
- R6: footprint (none) -> SAPR:R_0402_1005Metric; Manufacturer_Part_Number (none) -> RC0402FR-07110KL
- R7: footprint (none) -> SAPR:R_0805_2012Metric; Manufacturer_Part_Number (none) -> RC0805FR-072M32L
- R8: footprint (none) -> SAPR:R_0805_2012Metric; Manufacturer_Part_Number (none) -> RC0805FR-072M43L
- R9: footprint (none) -> SAPR:R_0402_1005Metric; Manufacturer_Part_Number (none) -> RC0402FR-07127KL
- VD1: Manufacturer_Part_Number (none) -> SS24FL
- VD2, VD3: footprint (none) -> SAPR:D_PowerDI-123; Manufacturer_Part_Number (none) -> DFLS240-7
- VD4: footprint (none) -> SAPR:D_SMA; Manufacturer_Part_Number (none) -> B230A-13-F
- XT1: footprint (none) -> SAPR:USB_Micro-B_Molex_47346-0001
Connections:
- net +15B: now also XT3.1; no longer C27.1, C32.1, DA7.1 (VOUT), R14.1
- net +16B: now also VD2.1; no longer VD2.
- net +3,3B: now also C10.1, XT3.4
- net +5B: now also XT3.2; no longer VD1.
- net -15B: now also C27.1, C32.1, DA7.1 (VOUT), R14.1, XT3.3
- net -16B: now also VD3.2; no longer VD3.
- net GND 2: now also C10.2, C11.2, C13.2, C14.2, C15.2, C18.2, C19.2, C20.2, DA2.17 (GND2), DA2.19 (EQ21), DA2.26 (GND2), DA4.2 (GND), R9.2, VD4.2, XT2.6, XT3.5, XT3.6; no longer VD4.
- net GND 3: now also R13.2; no longer DA3.21 (EP(AGND))
- net OTG_FS_DM: now also XT2.2
- net OTG_FS_DP: now also XT2.1
- net SUP_NEG_EN: now also DA3.11 (EN2), XT2.4
- net SUP_POS_EN: now also DA3.9 (EN1), XT2.5
- net UD_N: now also DA2.7 (UD-)
- net UN_P: now also DA2.8 (UD+)
- net at C28.2, DA5.6 (SW), L5.1: now also VD4.1; no longer VD4.
- net +1,8B: now reaches C13.1
- net +1,8B: now also C11.1, C14.1, C15.1, C18.1, C19.1, DA2.18 (V1P8V2), DA2.24 (VCC2), DA2.25 (V1P8V2)
- net VBUSIN: now reaches C1.1, DA2.1 (VBUS1), R1.1
- net VBUSIN: now also XT1.1
- net at R1.2: now also C7.1, DA2.5 (VCC1)
- net at DA3.2 (SW1), L2.2: now also VD2.2; no longer VD2.
- net at DA3.20 (SW2), L3.1: now also VD3.1; no longer VD3.
- net at C6.1, DA1.1 (+Vin): now also VD1.1; no longer VD1.
- new net +5_1B: VD1.2, XT2.3
- no-connect marks 9 -> 11
Other:
- moved on the sheet: C11, C13, C14, C15, C18, C19
